File: kicad/horizon.kicad_pcb (KiCad board)
At the start: 2 copper layers, 270 x 90 mm, 105 parts, among them J1 OLED, SW1 SW_Push, SW10 SW_Push, SW11 SW_Push, SW12 SW_Push, SW13 SW_Push, SW14 SW_Push, SW15 SW_Push, SW16 SW_Push, SW17 SW_Push, SW18 SW_Push, SW19 SW_Push, SW2 SW_Push, SW20 SW_Push, SW21 SW_Push, SW22 SW_Push, SW23 SW_Push, SW24 SW_Push, SW25 SW_Push, SW26 SW_Push, SW27 SW_Push, SW28 SW_Push, SW29 SW_Push, SW3 SW_Push, SW30 SW_Push, SW31 SW_Push, SW32 SW_Push, SW33 SW_Push, SW34 SW_Push, SW35 SW_Push, SW36 SW_Push, SW37 SW_Push, SW38 SW_Push, SW39 SW_Push, SW4 SW_Push, SW40 SW_Push, SW41 SW_Push, SW42 SW_Push, SW5 SW_Push, SW6 SW_Push, SW7 SW_Push, SW8 SW_Push, SW9 SW_Push, U1 PRO-MICRO

Commit message: Begin revision 2
Parts:
- removed the D25 at (280.0, 128.0)
- removed H10, H11, H12, H13, H14, H15, H9: Hole_Pad, horizon-footprints:MountingHole_M2
- removed R1, R2: R, horizon-footprints:R_0805
- added D1: D, horizon-footprints:D_SOD-123, F.Cu at (195.0, 115.0)
- D10: renamed from D28; footprint horizon-footprints:D_SOD-323 -> horizon-footprints:D_SOD-123; moved to F.Cu
- D11: renamed from D16; footprint horizon-footprints:D_SOD-323 -> horizon-footprints:D_SOD-123; moved to F.Cu
- D12: renamed from D4; footprint horizon-footprints:D_SOD-323 -> horizon-footprints:D_SOD-123; moved to F.Cu
- D13: renamed from D29; footprint horizon-footprints:D_SOD-323 -> horizon-footprints:D_SOD-123; moved to F.Cu
- D14: renamed from D17; footprint horizon-footprints:D_SOD-323 -> horizon-footprints:D_SOD-123; moved to F.Cu
- D15: renamed from D5; footprint horizon-footprints:D_SOD-323 -> horizon-footprints:D_SOD-123; moved to F.Cu
- D16: renamed from D30; footprint horizon-footprints:D_SOD-323 -> horizon-footprints:D_SOD-123; moved to F.Cu
- D17: renamed from D18; footprint horizon-footprints:D_SOD-323 -> horizon-footprints:D_SOD-123; moved to F.Cu
- D18: renamed from D6; footprint horizon-footprints:D_SOD-323 -> horizon-footprints:D_SOD-123; moved to F.Cu
- D19: renamed from D37; footprint horizon-footprints:D_SOD-323 -> horizon-footprints:D_SOD-123; moved to F.Cu
- D2: renamed from D13; footprint horizon-footprints:D_SOD-323 -> horizon-footprints:D_SOD-123; moved to F.Cu
- D20: renamed from D38; footprint horizon-footprints:D_SOD-323 -> horizon-footprints:D_SOD-123; moved to F.Cu
- D21: renamed from D39; footprint horizon-footprints:D_SOD-323 -> horizon-footprints:D_SOD-123; moved to F.Cu
- D22: renamed from D40; footprint horizon-footprints:D_SOD-323 -> horizon-footprints:D_SOD-123; moved to F.Cu
- D23: renamed from D41; footprint horizon-footprints:D_SOD-323 -> horizon-footprints:D_SOD-123; moved to F.Cu
- D24: renamed from D42; footprint horizon-footprints:D_SOD-323 -> horizon-footprints:D_SOD-123; moved to F.Cu
- D25: renamed from D12; footprint horizon-footprints:D_SOD-323 -> horizon-footprints:D_SOD-123; moved to F.Cu
- D26: renamed from D9; footprint horizon-footprints:D_SOD-323 -> horizon-footprints:D_SOD-123; moved to F.Cu
- D27: renamed from D33; footprint horizon-footprints:D_SOD-323 -> horizon-footprints:D_SOD-123; moved to F.Cu
- D28: renamed from D35; footprint horizon-footprints:D_SOD-323 -> horizon-footprints:D_SOD-123; moved to F.Cu
- D29: renamed from D23; footprint horizon-footprints:D_SOD-323 -> horizon-footprints:D_SOD-123; moved to F.Cu
- D3: renamed from D1; footprint horizon-footprints:D_SOD-323 -> horizon-footprints:D_SOD-123; moved to F.Cu
- D30: renamed from D20; footprint horizon-footprints:D_SOD-323 -> horizon-footprints:D_SOD-123; moved to F.Cu
- D31: renamed from D11; footprint horizon-footprints:D_SOD-323 -> horizon-footprints:D_SOD-123; moved to F.Cu
- D32: renamed from D8; footprint horizon-footprints:D_SOD-323 -> horizon-footprints:D_SOD-123; moved to F.Cu
- D33: renamed from D32; footprint horizon-footprints:D_SOD-323 -> horizon-footprints:D_SOD-123; moved to F.Cu
- D34: renamed from D36; footprint horizon-footprints:D_SOD-323 -> horizon-footprints:D_SOD-123; moved to F.Cu
- D35: renamed from D22; footprint horizon-footprints:D_SOD-323 -> horizon-footprints:D_SOD-123; moved to F.Cu
- D36: renamed from D7; footprint horizon-footprints:D_SOD-323 -> horizon-footprints:D_SOD-123; moved to F.Cu
- D37: renamed from D34; footprint horizon-footprints:D_SOD-323 -> horizon-footprints:D_SOD-123; moved to F.Cu
- D38: renamed from D24; footprint horizon-footprints:D_SOD-323 -> horizon-footprints:D_SOD-123; moved to F.Cu
- D39: renamed from D21; footprint horizon-footprints:D_SOD-323 -> horizon-footprints:D_SOD-123; moved to F.Cu
- D4: renamed from D26; footprint horizon-footprints:D_SOD-323 -> horizon-footprints:D_SOD-123; moved to F.Cu
- D40: renamed from D19; footprint horizon-footprints:D_SOD-323 -> horizon-footprints:D_SOD-123; moved to F.Cu
- D41: renamed from D10; footprint horizon-footprints:D_SOD-323 -> horizon-footprints:D_SOD-123; moved to F.Cu
- D42: renamed from D31; footprint horizon-footprints:D_SOD-323 -> horizon-footprints:D_SOD-123; moved to F.Cu
- D5: renamed from D14; footprint horizon-footprints:D_SOD-323 -> horizon-footprints:D_SOD-123; moved to F.Cu
- D6: renamed from D2; footprint horizon-footprints:D_SOD-323 -> horizon-footprints:D_SOD-123; moved to F.Cu
- D7: renamed from D27; footprint horizon-footprints:D_SOD-323 -> horizon-footprints:D_SOD-123; moved to F.Cu
- D8: renamed from D15; footprint horizon-footprints:D_SOD-323 -> horizon-footprints:D_SOD-123; moved to F.Cu
- D9: renamed from D3; footprint horizon-footprints:D_SOD-323 -> horizon-footprints:D_SOD-123; moved to F.Cu
- moved SW10 153.2 mm to (294.5, 104.5)
- moved SW11 153.2 mm to (313.5, 104.5)
- moved SW12 153.2 mm to (332.5, 104.5)
- moved SW25 153.2 mm to (85.5, 142.5)
- moved SW26 153.2 mm to (104.5, 142.5)
- moved SW27 153.2 mm to (123.5, 142.5)
- moved SW28 153.2 mm to (142.5, 142.5)
- moved SW29 153.2 mm to (161.5, 142.5)
- moved SW30 153.2 mm to (180.5, 142.5)
- moved SW7 153.2 mm to (237.5, 104.5)
- moved SW8 153.2 mm to (256.5, 104.5)
- moved SW9 153.2 mm to (275.5, 104.5)
- moved H2 142.2 mm to (223.0, 100.0)
- moved H7 128.4 mm to (323.0, 114.0)
- moved H6 114.8 mm to (95.0, 152.0)
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Connections:
- D10 pad 1: ROW5 -> ROW2
- D10 pad 2: Net-(D28-Pad2) -> Net-(D10-Pad2)
- D11 pad 1: ROW3 -> ROW2
- D11 pad 2: Net-(D16-Pad2) -> Net-(D11-Pad2)
- D12 pad 1: ROW1 -> ROW2
- D12 pad 2: Net-(D4-Pad2) -> Net-(D12-Pad2)
- D13 pad 1: ROW5 -> ROW3
- D13 pad 2: Net-(D29-Pad2) -> Net-(D13-Pad2)
- D14 pad 2: Net-(D17-Pad2) -> Net-(D14-Pad2)
- D15 pad 1: ROW1 -> ROW3
- D15 pad 2: Net-(D5-Pad2) -> Net-(D15-Pad2)
- D16 pad 1: ROW5 -> ROW3
- D16 pad 2: Net-(D30-Pad2) -> Net-(D16-Pad2)
- D17 pad 2: Net-(D18-Pad2) -> Net-(D17-Pad2)
- D18 pad 1: ROW1 -> ROW3
- D18 pad 2: Net-(D6-Pad2) -> Net-(D18-Pad2)
- D19 pad 1: ROW7 -> ROW4
- D19 pad 2: Net-(D37-Pad2) -> Net-(D19-Pad2)
- D2 pad 1: ROW3 -> ROW1
- D2 pad 2: Net-(D13-Pad2) -> Net-(D2-Pad2)
- D20 pad 1: ROW7 -> ROW4
- D20 pad 2: Net-(D38-Pad2) -> Net-(D20-Pad2)
- D21 pad 1: ROW7 -> ROW4
- D21 pad 2: Net-(D39-Pad2) -> Net-(D21-Pad2)
- D22 pad 1: ROW7 -> ROW4
- D22 pad 2: Net-(D40-Pad2) -> Net-(D22-Pad2)
- D23 pad 1: ROW7 -> ROW4
- D23 pad 2: Net-(D41-Pad2) -> Net-(D23-Pad2)
- D24 pad 1: ROW7 -> ROW4
- D24 pad 2: Net-(D42-Pad2) -> Net-(D24-Pad2)
- D25 pad 1: ROW2 -> ROW5
- D25 pad 2: Net-(D12-Pad2) -> Net-(D25-Pad2)
- D26 pad 1: ROW2 -> ROW5
- D26 pad 2: Net-(D9-Pad2) -> Net-(D26-Pad2)
- D27 pad 1: ROW6 -> ROW5
- D27 pad 2: Net-(D33-Pad2) -> Net-(D27-Pad2)
- D28 pad 1: ROW6 -> ROW5
- D28 pad 2: Net-(D35-Pad2) -> Net-(D28-Pad2)
- D29 pad 1: ROW4 -> ROW5
- D29 pad 2: Net-(D23-Pad2) -> Net-(D29-Pad2)
- D3 pad 2: Net-(D1-Pad2) -> Net-(D3-Pad2)
- D30 pad 1: ROW4 -> ROW5
- D30 pad 2: Net-(D20-Pad2) -> Net-(D30-Pad2)
- D31 pad 1: ROW2 -> ROW6
- D31 pad 2: Net-(D11-Pad2) -> Net-(D31-Pad2)
- D32 pad 1: ROW2 -> ROW6
- D32 pad 2: Net-(D8-Pad2) -> Net-(D32-Pad2)
- D33 pad 2: Net-(D32-Pad2) -> Net-(D33-Pad2)
- D34 pad 2: Net-(D36-Pad2) -> Net-(D34-Pad2)
- D35 pad 1: ROW4 -> ROW6
- D35 pad 2: Net-(D22-Pad2) -> Net-(D35-Pad2)
- D36 pad 1: ROW2 -> ROW6
- D36 pad 2: Net-(D7-Pad2) -> Net-(D36-Pad2)
- D37 pad 1: ROW6 -> ROW7
- D37 pad 2: Net-(D34-Pad2) -> Net-(D37-Pad2)
- D38 pad 1: ROW4 -> ROW7
- D38 pad 2: Net-(D24-Pad2) -> Net-(D38-Pad2)
- D39 pad 1: ROW4 -> ROW7
- D39 pad 2: Net-(D21-Pad2) -> Net-(D39-Pad2)
- D4 pad 1: ROW5 -> ROW1
- D4 pad 2: Net-(D26-Pad2) -> Net-(D4-Pad2)
- D40 pad 1: ROW4 -> ROW7
- D40 pad 2: Net-(D19-Pad2) -> Net-(D40-Pad2)
- D41 pad 1: ROW2 -> ROW7
- D41 pad 2: Net-(D10-Pad2) -> Net-(D41-Pad2)
- D42 pad 1: ROW6 -> ROW7
- D42 pad 2: Net-(D31-Pad2) -> Net-(D42-Pad2)
- D5 pad 1: ROW3 -> ROW1
- D5 pad 2: Net-(D14-Pad2) -> Net-(D5-Pad2)
- D6 pad 2: Net-(D2-Pad2) -> Net-(D6-Pad2)
- D7 pad 1: ROW5 -> ROW2
- D7 pad 2: Net-(D27-Pad2) -> Net-(D7-Pad2)
- D8 pad 1: ROW3 -> ROW2
- D8 pad 2: Net-(D15-Pad2) -> Net-(D8-Pad2)
- D9 pad 1: ROW1 -> ROW2
- D9 pad 2: Net-(D3-Pad2) -> Net-(D9-Pad2)
- U1 pad 10: ROW5 -> COL4
- U1 pad 11: ROW6 -> COL5
- U1 pad 12: ROW7 -> COL6
- U1 pad 13: ROW2 -> ROW7
- U1 pad 14: ROW1 -> ROW6
- U1 pad 15: COL6 -> ROW4
- U1 pad 16: COL5 -> ROW2
- U1 pad 17: COL4 -> ROW5
- U1 pad 18: COL3 -> ROW3
- U1 pad 19: COL2 -> ROW1
- U1 pad 20: COL1 -> (no net)
- U1 pad 7: (no net) -> COL1
- U1 pad 8: ROW3 -> COL2
- U1 pad 9: ROW4 -> COL3
Routing:
- net ROW3: track 117.7 -> 16.5 mm
- net Net-(D36-Pad2): track 48.5 -> 120.3 mm
- net Net-(D12-Pad2): track 48.5 -> 119.2 mm
- net Net-(D1-Pad2): track 43.4 -> 114.1 mm
- net Net-(D35-Pad2): track 32.0 -> 102.5 mm
- net Net-(D34-Pad2): track 16.4 -> 84.7 mm
- net Net-(D25-Pad2): track 43.4 -> 111.3 mm
- net Net-(D2-Pad2): track 26.9 -> 93.5 mm
- net Net-(D11-Pad2): track 32.0 -> 98.6 mm
- net Net-(D26-Pad2): track 26.9 -> 93.5 mm
- net Net-(D13-Pad2): track 43.4 -> 108.7 mm
- net Net-(D24-Pad2): track 48.5 -> 113.4 mm
- net Net-(D27-Pad2): track 10.8 -> 75.7 mm
- net Net-(D14-Pad2): track 26.9 -> 90.5 mm
- net Net-(D23-Pad2): track 32.0 -> 95.6 mm
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Other:
- board size 270 x 90 mm -> 266 x 76 mm
- board text added: "rev2"
- board text removed: "rev1"

Commit message: Create bottom plate board. Begin laying out Choc switch board. Clean up footprints and remove unused ones
Parts:
- H1, H2, H3, H4, H5, H6, H7, H8: footprint horizon-footprints:MountingHole_M2 -> horizon-footprints:Mount_M2
- J1: footprint horizon-footprints:Header_THT_1x04_2.54mm -> horizon-footprints:Header_1x04_2.54mm
- TSW1: footprint horizon-footprints:SW_PUSH_6mm -> horizon-footprints:SW_Push_6mm
- moved LOGO1 43.0 mm to (209.0, 147.0)
Routing:
- net COL1: track 343.1 -> 342.2 mm

Commit message: Adjust center component layout for MX and Choc consistency.
Parts:
- LOGO1: moved to F.Cu
- moved LOGO1 9.00 mm to (209.0, 138.0), turned to 0 degrees
- moved TSW1 8.50 mm to (209.0, 147.0), turned to 90 degrees
- moved D37 4.50 mm to (199.5, 147.0)
- moved D38 4.50 mm to (201.5, 147.0)
- moved D39 4.50 mm to (203.5, 147.0)
- moved D40 4.50 mm to (214.5, 147.0)
- moved D41 4.50 mm to (216.5, 147.0)
- moved D42 4.50 mm to (218.5, 147.0)
- moved D1 1.50 mm to (195.0, 116.5)
- moved D10 1.50 mm to (223.0, 112.5)
- moved D11 1.50 mm to (223.0, 114.5)
- moved D12 1.50 mm to (223.0, 116.5)
- moved D2 1.50 mm to (195.0, 114.5)
- moved D25 1.50 mm to (195.0, 140.5)
- moved D26 1.50 mm to (195.0, 138.5)
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Connections:
- U1 pad 1: (no net) -> ROW2
- U1 pad 15: ROW4 -> ROW5
- U1 pad 16: ROW2 -> ROW3
- U1 pad 17: ROW5 -> ROW1
- U1 pad 18: ROW3 -> (no net)
- U1 pad 19: ROW1 -> (no net)
- U1 pad 2: (no net) -> ROW4
Routing:
- net COL1: track 342.2 -> 0.00 mm
- net COL2: track 338.4 -> 0.00 mm
- net COL3: track 334.6 -> 0.00 mm
- net COL4: track 330.7 -> 0.00 mm
- net COL5: track 326.9 -> 0.00 mm
- net COL6: track 322.3 -> 0.00 mm
- net Net-(D36-Pad2): track 120.4 -> 0.00 mm
- net Net-(D12-Pad2): track 119.2 -> 0.00 mm
- net Net-(D1-Pad2): track 114.1 -> 0.00 mm
- net Net-(D24-Pad2): track 113.4 -> 0.00 mm
- net Net-(D25-Pad2): track 111.4 -> 0.00 mm
- net Net-(D13-Pad2): track 108.3 -> 0.00 mm
- net Net-(D35-Pad2): track 102.5 -> 0.00 mm
- net Net-(D11-Pad2): track 98.6 -> 0.00 mm
- net Net-(D23-Pad2): track 95.6 -> 0.00 mm
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
Commit message: Use 50 key layout on MX version
Parts:
- removed the D1 at (195.0, 116.5)
- removed the D13 at (195.0, 118.5)
- removed the D19 at (223.0, 128.5)
- removed the D20 at (223.0, 126.5)
- removed the D25 at (195.0, 140.5)
- removed the D31 at (223.0, 130.5)
- removed the D32 at (223.0, 132.5)
- removed the D37 at (199.5, 147.0)
- removed the D7 at (223.0, 106.5)
- removed the D8 at (223.0, 108.5)
- removed the SW1 at (85.5, 104.5)
- removed the SW13 at (85.5, 123.5)
- removed the SW19 at (237.5, 123.5)
- removed the SW20 at (256.5, 123.5)
- removed the SW25 at (85.5, 142.5)
- removed the SW31 at (237.5, 142.5)
- removed the SW32 at (256.5, 142.5)
- removed the SW37 at (161.5, 161.5)
- removed the SW7 at (237.5, 104.5)
- removed the SW8 at (256.5, 104.5)
- added D11: D, horizon-footprints:D_SOD-123, F.Cu at (223.5, 112.5)
- added D12: D, horizon-footprints:D_SOD-123, F.Cu at (223.5, 114.5)
- added D18: D, horizon-footprints:D_SOD-123, F.Cu at (194.5, 126.5)
- added D23: D, horizon-footprints:D_SOD-123, F.Cu at (223.5, 118.5)
- added D24: D, horizon-footprints:D_SOD-123, F.Cu at (223.5, 116.5)
- added D30: D, horizon-footprints:D_SOD-123, F.Cu at (194.5, 128.5)
- added D35: D, horizon-footprints:D_SOD-123, F.Cu at (223.5, 136.5)
- added D36: D, horizon-footprints:D_SOD-123, F.Cu at (223.5, 138.5)
- added D42: D, horizon-footprints:D_SOD-123, F.Cu at (206.0, 147.5)
- added D43: D, horizon-footprints:D_SOD-123, F.Cu at (208.0, 147.5)
- added D44: D, horizon-footprints:D_SOD-123, F.Cu at (210.0, 147.5)
- added D45: D, horizon-footprints:D_SOD-123, F.Cu at (212.0, 147.5)
- added D46: D, horizon-footprints:D_SOD-123, F.Cu at (214.0, 147.5)
- added D47: D, horizon-footprints:D_SOD-123, F.Cu at (216.0, 147.5)
- added D48: D, horizon-footprints:D_SOD-123, F.Cu at (218.0, 147.5)
- added D49: D, horizon-footprints:D_SOD-123, F.Cu at (223.5, 142.5)
- added D50: D, horizon-footprints:D_SOD-123, F.Cu at (223.5, 140.5)
- added D6: D, horizon-footprints:D_SOD-123, F.Cu at (194.5, 104.5)
- added SW11: SW_Push, horizon-footprints:SW_MX, F.Cu at (313.5, 104.5)
- added SW12: SW_Push, horizon-footprints:SW_MX, F.Cu at (332.5, 104.5)
- added SW18: SW_Push, horizon-footprints:SW_MX, F.Cu at (180.5, 123.5)
- added SW23: SW_Push, horizon-footprints:SW_MX, F.Cu at (313.5, 123.5)
- added SW24: SW_Push, horizon-footprints:SW_MX, F.Cu at (332.5, 123.5)
- added SW30: SW_Push, horizon-footprints:SW_MX, F.Cu at (180.5, 142.5)
- added SW35: SW_Push, horizon-footprints:SW_MX, F.Cu at (313.5, 142.5)
- added SW36: SW_Push, horizon-footprints:SW_MX, F.Cu at (332.5, 142.5)
- added SW42: SW_Push, horizon-footprints:SW_MX, F.Cu at (180.5, 161.5)
- added SW43: SW_Push, horizon-footprints:SW_MX, F.Cu at (199.5, 161.5)
- added SW44: SW_Push, horizon-footprints:SW_MX, F.Cu at (218.5, 161.5)
- added SW45: SW_Push, horizon-footprints:SW_MX, F.Cu at (237.5, 161.5)
- added SW46: SW_Push, horizon-footprints:SW_MX, F.Cu at (256.5, 161.5)
- added SW47: SW_Push, horizon-footprints:SW_MX, F.Cu at (275.5, 161.5)
- added SW48: SW_Push, horizon-footprints:SW_MX, F.Cu at (294.5, 161.5)
- added SW49: SW_Push, horizon-footprints:SW_MX, F.Cu at (313.5, 161.5)
- added SW50: SW_Push, horizon-footprints:SW_MX, F.Cu at (332.5, 161.5)
- added SW6: SW_Push, horizon-footprints:SW_MX, F.Cu at (180.5, 104.5)
- LOGO1: moved to B.Cu
- moved SW37 95.0 mm to (85.5, 161.5)
- moved SW38 95.0 mm to (104.5, 161.5)
- moved SW39 95.0 mm to (123.5, 161.5)
- moved SW40 95.0 mm to (142.5, 161.5)
- moved SW41 95.0 mm to (161.5, 161.5)
- moved SW10 38.0 mm to (294.5, 104.5)
- moved SW19 38.0 mm to (237.5, 123.5)
- moved SW20 38.0 mm to (256.5, 123.5)
- moved SW21 38.0 mm to (275.5, 123.5)
- moved SW22 38.0 mm to (294.5, 123.5)
- moved SW31 38.0 mm to (237.5, 142.5)
- moved SW32 38.0 mm to (256.5, 142.5)
- moved SW33 38.0 mm to (275.5, 142.5)
- moved SW34 38.0 mm to (294.5, 142.5)
- moved SW7 38.0 mm to (237.5, 104.5)
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- renumbered D2 to D1, D12 to D10, D14 to D13, D15 to D14, D16 to D15, D17 to D16, D18 to D17, D21 to D19, D3 to D2, D22 to D20, D23 to D21, D24 to D22, D26 to D25, D27 to D26, D28 to D27, D29 to D28, D30 to D29, D4 to D3, D33 to D31, D34 to D32, D35 to D33, D36 to D34, D38 to D37, D39 to D38, D40 to D39, D5 to D4, D41 to D40, D42 to D41, D6 to D5, D9 to D7, D10 to D8, D11 to D9, SW2 to SW1, SW12 to SW10, SW14 to SW13, SW15 to SW14, SW16 to SW15, SW17 to SW16, SW18 to SW17, SW21 to SW19, SW3 to SW2, SW22 to SW20, SW23 to SW21, SW24 to SW22, SW26 to SW25, SW27 to SW26, SW28 to SW27, SW29 to SW28, SW30 to SW29, SW4 to SW3, SW33 to SW31, SW34 to SW32, SW35 to SW33, SW36 to SW34, SW38 to SW37, SW39 to SW38, SW40 to SW39, SW5 to SW4, SW41 to SW40, SW42 to SW41, SW6 to SW5, SW9 to SW7, SW10 to SW8, SW11 to SW9
Connections:
- SW1 pad 1: COL2 -> COL1
- SW10 pad 1: COL6 -> COL5
- SW13 pad 1: COL2 -> COL1
- SW14 pad 1: COL3 -> COL2
- SW15 pad 1: COL4 -> COL3
- SW16 pad 1: COL5 -> COL4
- SW17 pad 1: COL6 -> COL5
- SW19 pad 1: COL3 -> COL2
- SW2 pad 1: COL3 -> COL2
- SW20 pad 1: COL4 -> COL3
- SW21 pad 1: COL5 -> COL4
- SW22 pad 1: COL6 -> COL5
- SW25 pad 1: COL2 -> COL1
- SW26 pad 1: COL3 -> COL2
- SW27 pad 1: COL4 -> COL3
- SW28 pad 1: COL5 -> COL4
- SW29 pad 1: COL6 -> COL5
- SW3 pad 1: COL4 -> COL3
- SW31 pad 1: COL3 -> COL2
- SW32 pad 1: COL4 -> COL3
- SW33 pad 1: COL5 -> COL4
- SW34 pad 1: COL6 -> COL5
- SW37 pad 1: COL2 -> COL1
- SW38 pad 1: COL3 -> COL2
- SW39 pad 1: COL4 -> COL3
- SW4 pad 1: COL5 -> COL4
- SW40 pad 1: COL5 -> COL4
- SW41 pad 1: COL6 -> COL5
- SW5 pad 1: COL6 -> COL5
- SW7 pad 1: COL3 -> COL2
- SW8 pad 1: COL4 -> COL3
- SW9 pad 1: COL5 -> COL4
- U1 pad 10: COL4 -> ROW6
- U1 pad 11: COL5 -> ROW7
- U1 pad 12: COL6 -> ROW8
- U1 pad 13: ROW7 -> COL7
- U1 pad 14: ROW6 -> COL6
- U1 pad 15: ROW5 -> COL5
- U1 pad 16: ROW3 -> COL4
- U1 pad 17: ROW1 -> COL3
- U1 pad 18: (no net) -> COL2
- U1 pad 19: (no net) -> COL1
- U1 pad 20: (no net) -> ROW1
- U1 pad 7: COL1 -> (no net)
- U1 pad 8: COL2 -> ROW3
- U1 pad 9: COL3 -> ROW5
Routing:
- net COL2: track 0.00 -> 277.9 mm
- net COL3: track 0.00 -> 274.1 mm
- net COL4: track 0.00 -> 270.3 mm
- net COL5: track 0.00 -> 266.4 mm
- net COL6: track 0.00 -> 262.6 mm
- net COL1: track 0.00 -> 258.7 mm
- net COL7: track 0.00 -> 226.1 mm
- net Net-(D36-Pad2): track 0.00 -> 122.8 mm
- net Net-(D12-Pad2): track 0.00 -> 121.3 mm
- net Net-(D50-Pad2): track 0.00 -> 117.3 mm
- net Net-(D25-Pad2): track 0.00 -> 113.8 mm
- net Net-(D37-Pad2): track 0.00 -> 113.2 mm
- net Net-(D1-Pad2): track 0.00 -> 112.7 mm
- net Net-(D24-Pad2): track 0.00 -> 112.0 mm
- net Net-(D13-Pad2): track 0.00 -> 106.9 mm
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
Commit message: Clean up MX version before overhaul
Parts:
- removed H5, H6, H7, H8: Hole_Pad, horizon-footprints:Mount_M2
- RESET1: renamed from TSW1; value RESET -> SW_Push
- U1: value PRO-MICRO -> Pro-Micro
- moved H1 0.71 mm to (195.0, 100.0)
- moved H2 0.71 mm to (223.0, 100.0)
- moved H3 0.71 mm to (195.0, 147.0)
- moved H4 0.71 mm to (223.0, 147.0)
- moved D1 0.50 mm to (195.0, 114.5)
- moved D10 0.50 mm to (223.0, 110.5)
- moved D11 0.50 mm to (223.0, 112.5)
- moved D12 0.50 mm to (223.0, 114.5)
- moved D13 0.50 mm to (195.0, 116.5)
- moved D14 0.50 mm to (195.0, 118.5)
- moved D15 0.50 mm to (195.0, 120.5)
- moved D16 0.50 mm to (195.0, 122.5)
- moved D17 0.50 mm to (195.0, 124.5)
- moved D18 0.50 mm to (195.0, 126.5)
- moved D19 0.50 mm to (223.0, 126.5)
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Routing:
- net Net-(RESET1-Pad1): track 47.7 -> 43.2 mm
- net COL1: track 258.7 -> 257.1 mm
- net ROW8: track 38.1 -> 36.8 mm
- net ROW7: track 42.0 -> 40.8 mm
- net ROW3: track 70.7 -> 69.5 mm
- net ROW5: track 57.4 -> 56.2 mm
- net ROW2: track 18.6 -> 17.4 mm
- net ROW4: track 27.1 -> 27.6 mm
- net Net-(D18-Pad2): track 17.1 -> 17.6 mm
- net ROW1: track 18.5 -> 18.0 mm
- net Net-(D9-Pad2): track 60.2 -> 60.7 mm
- net Net-(D8-Pad2): track 40.6 -> 41.1 mm
- net Net-(D7-Pad2): track 17.0 -> 17.5 mm
- net Net-(D6-Pad2): track 11.9 -> 12.4 mm
- net Net-(D50-Pad2): track 117.3 -> 117.8 mm
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
Commit message: Layout MX PCB
Parts:
- removed J1: OLED, horizon-footprints:Header_1x04_2.54mm
- removed RESET1: SW_Push, horizon-footprints:SW_Push_6mm
- added BTN1: RESET, horizon-footprints:SW_Push_6mm, F.Cu at (195.0, 117.0)
- added D51: D, horizon-footprints:D_SOD-123, B.Cu at (313.5, 166.2)
- added D52: D, horizon-footprints:D_SOD-123, B.Cu at (332.5, 166.2)
- added H5: Hole_Pad, horizon-footprints:Mount_M2, F.Cu at (195.0, 100.0)
- added H6: Hole_Pad, horizon-footprints:Mount_M2, F.Cu at (223.0, 100.0)
- added H7: Hole_Pad, horizon-footprints:Mount_M2, F.Cu at (195.0, 128.0)
- added H8: Hole_Pad, horizon-footprints:Mount_M2, F.Cu at (223.0, 128.0)
- added SS1: POWER, horizon-footprints:SS12D00, F.Cu at (195.0, 110.0)
- added SW51: SW_Push, horizon-footprints:SW_MX, F.Cu at (313.5, 161.5)
- added SW52: SW_Push, horizon-footprints:SW_MX, F.Cu at (332.5, 161.5)
- added TB1: BATTERY, horizon-footprints:KF350-2P, F.Cu at (223.0, 114.0)
- D1, D10, D11, D12, D13, D14, D15, D16, D17, D18, D19, D2, D20, D21, D22, D23, D24, D25, D26, D27, D28, D29, D3, D30, D31, D32, D33, D34, D35, D36, D37, D38, D39, D4, D40, D41, D42, D43, D44, D45, D46, D47, D48, D49, D5, D50, D6, D7, D8, D9: moved to B.Cu
- LOGO1: footprint horizon-footprints:Logo_Horizon -> horizon-footprints:Logo_Horizon_Small
- U1: value Pro-Micro -> PRO-MICRO
- moved SW37 228.8 mm to (313.5, 142.5)
- moved SW38 228.8 mm to (332.5, 142.5)
- moved D38 137.6 mm to (332.5, 147.2), turned to 0 degrees
- moved D37 118.7 mm to (313.5, 147.2), turned to 0 degrees
- moved D39 116.1 mm to (85.5, 166.2), turned to 0 degrees
- moved D13 110.1 mm to (85.5, 128.2), turned to 0 degrees
- moved D24 110.1 mm to (332.5, 128.2)
- moved D25 109.8 mm to (85.5, 147.2), turned to 0 degrees
- moved D1 109.6 mm to (85.5, 109.2), turned to 0 degrees
- moved D12 109.6 mm to (332.5, 109.2)
- moved H1 101.0 mm to (95.0, 114.0)
- moved H2 101.0 mm to (323.0, 114.0)
- moved H3 100.1 mm to (95.0, 152.0)
- moved H4 100.1 mm to (323.0, 152.0)
- moved D40 99.4 mm to (104.5, 166.2), turned to 0 degrees
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Connections:
- D10 pad 1: ROW2 -> ROW1
- D11 pad 1: ROW2 -> ROW1
- D12 pad 1: ROW2 -> ROW1
- D13 pad 1: ROW3 -> ROW2
- D14 pad 1: ROW3 -> ROW2
- D15 pad 1: ROW3 -> ROW2
- D16 pad 1: ROW3 -> ROW2
- D17 pad 1: ROW3 -> ROW2
- D18 pad 1: ROW3 -> ROW2
- D19 pad 1: ROW4 -> ROW2
- D20 pad 1: ROW4 -> ROW2
- D21 pad 1: ROW4 -> ROW2
- D22 pad 1: ROW4 -> ROW2
- D23 pad 1: ROW4 -> ROW2
- D24 pad 1: ROW4 -> ROW2
- D25 pad 1: ROW5 -> ROW3
- D26 pad 1: ROW5 -> ROW3
- D27 pad 1: ROW5 -> ROW3
- D28 pad 1: ROW5 -> ROW3
- D29 pad 1: ROW5 -> ROW3
- D30 pad 1: ROW5 -> ROW3
- D31 pad 1: ROW6 -> ROW3
- D32 pad 1: ROW6 -> ROW3
- D33 pad 1: ROW6 -> ROW3
- D34 pad 1: ROW6 -> ROW3
- D35 pad 1: ROW6 -> ROW3
- D36 pad 1: ROW6 -> ROW3
- D37 pad 1: ROW7 -> ROW3
- D38 pad 1: ROW7 -> ROW3
- D39 pad 1: ROW7 -> ROW4
- D40 pad 1: ROW7 -> ROW4
- D41 pad 1: ROW7 -> ROW4
- D42 pad 1: ROW7 -> ROW4
- D43 pad 1: ROW7 -> ROW4
- D44 pad 1: ROW8 -> ROW4
- D45 pad 1: ROW8 -> ROW4
- D46 pad 1: ROW8 -> ROW4
- D47 pad 1: ROW8 -> ROW4
- D48 pad 1: ROW8 -> ROW4
- D49 pad 1: ROW8 -> ROW4
- D50 pad 1: ROW8 -> ROW4
- D7 pad 1: ROW2 -> ROW1
- D8 pad 1: ROW2 -> ROW1
- D9 pad 1: ROW2 -> ROW1
- SW10 pad 1: COL5 -> COL12
- SW11 pad 1: COL6 -> COL13
- SW12 pad 1: COL7 -> COL14
- SW19 pad 1: COL2 -> COL9
- SW20 pad 1: COL3 -> COL10
- SW21 pad 1: COL4 -> COL11
- SW22 pad 1: COL5 -> COL12
- SW23 pad 1: COL6 -> COL13
- SW24 pad 1: COL7 -> COL14
- SW31 pad 1: COL2 -> COL7
- SW32 pad 1: COL3 -> COL8
- SW33 pad 1: COL4 -> COL9
- SW34 pad 1: COL5 -> COL10
- SW35 pad 1: COL6 -> COL11
- SW36 pad 1: COL7 -> COL12
- SW37 pad 1: COL1 -> COL13
- SW38 pad 1: COL2 -> COL14
- SW39 pad 1: COL3 -> COL1
- SW40 pad 1: COL4 -> COL2
- SW41 pad 1: COL5 -> COL3
- SW42 pad 1: COL6 -> COL4
- SW43 pad 1: COL7 -> COL5
- SW44 pad 1: COL1 -> COL6
- SW45 pad 1: COL2 -> COL7
- SW46 pad 1: COL3 -> COL8
- SW47 pad 1: COL4 -> COL9
- SW48 pad 1: COL5 -> COL10
- SW49 pad 1: COL6 -> COL11
- SW50 pad 1: COL7 -> COL12
- SW7 pad 1: COL2 -> COL9
- SW8 pad 1: COL3 -> COL10
- SW9 pad 1: COL4 -> COL11
- U1 pad 1: ROW2 -> ROW1
- U1 pad 10: ROW6 -> COL10
- U1 pad 11: ROW7 -> COL9
- U1 pad 12: ROW8 -> COL8
- U1 pad 2: ROW4 -> ROW2
- U1 pad 20: ROW1 -> ROW4
- U1 pad 21: VCC -> (no net)
- U1 pad 22: Net-(RESET1-Pad1) -> RESET
- U1 pad 24: (no net) -> RAW
- U1 pad 5: SDA -> ROW3
- U1 pad 6: SCL -> COL14
- U1 pad 7: (no net) -> COL13
- U1 pad 8: ROW3 -> COL12
- U1 pad 9: ROW5 -> COL11
Routing:
- net ROW4: track 27.6 -> 334.0 mm, vias 0 -> 1
- net ROW2: track 17.4 -> 302.0 mm
- net ROW1: track 18.0 -> 277.9 mm
- net ROW3: track 69.5 -> 315.0 mm, vias 0 -> 1
- net COL7: track 226.1 -> 34.3 mm
- net COL14: track 0.00 -> 185.1 mm
- net COL6: track 262.6 -> 88.1 mm
- net COL13: track 0.00 -> 163.9 mm
- net COL5: track 266.4 -> 108.2 mm
- net COL12: track 0.00 -> 142.8 mm
- net COL4: track 270.3 -> 129.3 mm
- net COL3: track 274.1 -> 150.4 mm
- net COL11: track 0.00 -> 121.7 mm
- net Net-(D36-Pad2): track 123.3 -> 10.1 mm
- net Net-(D12-Pad2): track 121.8 -> 10.1 mm
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Other:
- board text added: "rev2 | MX"
- board text removed: "rev2"
