File: kicad/choc/horizon-choc.kicad_pcb (KiCad board)
At the start: 2 copper layers, 252 x 68 mm, 116 parts, among them SW1 SW_Push, SW10 SW_Push, SW11 SW_Push, SW12 SW_Push, SW13 SW_Push, SW14 SW_Push, SW15 SW_Push, SW16 SW_Push, SW17 SW_Push, SW18 SW_Push, SW19 SW_Push, SW2 SW_Push, SW20 SW_Push, SW21 SW_Push, SW22 SW_Push, SW23 SW_Push, SW24 SW_Push, SW25 SW_Push, SW26 SW_Push, SW27 SW_Push, SW28 SW_Push, SW29 SW_Push, SW3 SW_Push, SW30 SW_Push, SW31 SW_Push, SW32 SW_Push, SW33 SW_Push, SW34 SW_Push, SW35 SW_Push, SW36 SW_Push, SW37 SW_Push, SW38 SW_Push, SW39 SW_Push, SW4 SW_Push, SW40 SW_Push, SW41 SW_Push, SW42 SW_Push, SW43 SW_Push, SW44 SW_Push, SW45 SW_Push, SW46 SW_Push, SW47 SW_Push, SW48 SW_Push, SW49 SW_Push, SW5 SW_Push, SW50 SW_Push, SW51 SW_Push, SW52 SW_Push, SW6 SW_Push, SW7 SW_Push, SW8 SW_Push, SW9 SW_Push, U1 PRO-MICRO

Commit message: Update projects to KiCad 6 and regenerate gerbers
Other:
- rule pad_to_mask_clearance: 0 -> 0.051

Commit message: Upgrade revision to 2.3. Remove KiCad 5 files
Other:
- board text added: "rev2.3 | Choc"
- board text removed: "rev2.2 | Choc"
Changed lines of the file:
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@@
   (title_block
     (title "Horizon Choc")
-    (date "2021-10-25")
-    (rev "2.2")
+    (date "2022-03-21")
+    (rev "2.3")
     (company "skarrmann")
   )
@@
     (effects (font (size 1 1) (thickness 0.15)) (justify mirror))
   )
-  (gr_text "rev2.2 | Choc" (at 148 91.5) (layer "B.SilkS")
+  (gr_text "rev2.3 | Choc" (at 148 91.5) (layer "B.SilkS")
     (effects (font (size 1 1) (thickness 0.15)) (justify mirror))
   )

Commit message: Upgrade plugin and project files to KiCad 7
Other:
- board text added: "rev2.4 | Choc"
- board text removed: "rev2.3 | Choc"
