File: kicad/mx/horizon-mx.kicad_pcb (KiCad board)
At the start: 2 copper layers, 266 x 76 mm, 116 parts, among them SW1 SW_Push, SW10 SW_Push, SW11 SW_Push, SW12 SW_Push, SW13 SW_Push, SW14 SW_Push, SW15 SW_Push, SW16 SW_Push, SW17 SW_Push, SW18 SW_Push, SW19 SW_Push, SW2 SW_Push, SW20 SW_Push, SW21 SW_Push, SW22 SW_Push, SW23 SW_Push, SW24 SW_Push, SW25 SW_Push, SW26 SW_Push, SW27 SW_Push, SW28 SW_Push, SW29 SW_Push, SW3 SW_Push, SW30 SW_Push, SW31 SW_Push, SW32 SW_Push, SW33 SW_Push, SW34 SW_Push, SW35 SW_Push, SW36 SW_Push, SW37 SW_Push, SW38 SW_Push, SW39 SW_Push, SW4 SW_Push, SW40 SW_Push, SW41 SW_Push, SW42 SW_Push, SW43 SW_Push, SW44 SW_Push, SW45 SW_Push, SW46 SW_Push, SW47 SW_Push, SW48 SW_Push, SW49 SW_Push, SW5 SW_Push, SW50 SW_Push, SW51 SW_Push, SW52 SW_Push, SW6 SW_Push, SW7 SW_Push, SW8 SW_Push, SW9 SW_Push, U1 PRO-MICRO

Commit message: Upgrade revision to 2.3. Remove KiCad 5 files
Routing:
- net COL5: track 108.2 -> 111.0 mm
- net COL4: track 129.3 -> 132.2 mm
- net COL2: track 171.6 -> 174.4 mm
- net COL13: track 163.9 -> 166.8 mm
- net COL9: track 83.5 -> 86.3 mm
- net COL6: track 88.1 -> 91.0 mm
- net COL10: track 100.6 -> 103.4 mm
- net COL3: track 150.4 -> 153.3 mm
- net COL12: track 142.8 -> 145.7 mm
- net COL11: track 121.7 -> 124.5 mm
- net COL1: track 192.7 -> 195.5 mm
- net COL14: track 185.1 -> 187.9 mm
- net COL8: track 32.8 -> 33.7 mm
- net COL7: track 34.3 -> 35.3 mm
Other:
- board text added: "rev2.3 | MX"
- board text removed: "rev2.2 | MX"

Commit message: Upgrade plugin and project files to KiCad 7
Other:
- board text added: "rev2.4 | MX"
- board text removed: "rev2.3 | MX"
